Commit message: update the robot

File: install/farm_robot_description/share/farm_robot_description/urdf/farm_bot.xacro (robot description, xacro)
@@ -1,154 +1 @@
-<?xml version="1.0"?>
-<robot xmlns:xacro="http://www.ros.org/wiki/xacro" name="farm_bot">
-  <!-- Basic dimensions -->
-  <xacro:property name="wheel_radius" value="0.08"/>
-  <xacro:property name="wheel_width" value="0.03"/>
-  <xacro:property name="chassis_length" value="0.40"/>
-  <xacro:property name="chassis_width" value="0.30"/>
-  <xacro:property name="chassis_height" value="0.12"/>
-  <xacro:property name="wheel_sep" value="${chassis_width}"/>
-  <!-- Base link -->
-  <link name="base_link">
-    <inertial>
-      <origin xyz="0 0 0"/>
-      <mass value="8.0"/>
-      <inertia ixx="0.2" ixy="0" ixz="0" iyy="0.2" iyz="0" izz="0.2"/>
-    </inertial>
-    <visual>
-      <origin xyz="0 0 ${chassis_height/2}"/>
-      <geometry>
-        <box size="${chassis_length} ${chassis_width} ${chassis_height}"/>
-      </geometry>
-      <material name="grey">
-        <color rgba="0.6 0.6 0.6 1.0"/>
-      </material>
-    </visual>
-    <collision>
-      <origin xyz="0 0 ${chassis_height/2}"/>
-      <geometry>
-        <box size="${chassis_length} ${chassis_width} ${chassis_height}"/>
-      </geometry>
-    </collision>
-  </link>
-  <!-- Wheels -->
-  <link name="left_wheel">
-    <visual>
-      <origin rpy="0 1.5708 0"/>
-      <geometry>
-        <cylinder length="${wheel_width}" radius="${wheel_radius}"/>
-      </geometry>
-      <material name="black">
-        <color rgba="0.1 0.1 0.1 1.0"/>
-      </material>
-    </visual>
-    <collision>
-      <origin rpy="0 1.5708 0"/>
-      <geometry>
-        <cylinder length="${wheel_width}" radius="${wheel_radius}"/>
-      </geometry>
-    </collision>
-    <inertial>
-      <mass value="0.5"/>
-      <inertia ixx="0.01" ixy="0" ixz="0" iyy="0.01" iyz="0" izz="0.01"/>
-    </inertial>
-  </link>
-  <link name="right_wheel">
-    <visual>
-      <origin rpy="0 1.5708 0"/>
-      <geometry>
-        <cylinder length="${wheel_width}" radius="${wheel_radius}"/>
-      </geometry>
-      <material name="black">
-        <color rgba="0.1 0.1 0.1 1.0"/>
-      </material>
-    </visual>
-    <collision>
-      <origin rpy="0 1.5708 0"/>
-      <geometry>
-        <cylinder length="${wheel_width}" radius="${wheel_radius}"/>
-      </geometry>
-    </collision>
-    <inertial>
-      <mass value="0.5"/>
-      <inertia ixx="0.01" ixy="0" ixz="0" iyy="0.01" iyz="0" izz="0.01"/>
-    </inertial>
-  </link>
-  <!-- Camera -->
-  <link name="camera_link">
-    <visual>
-      <origin xyz="${chassis_length/2 - 0.1} 0 ${chassis_height + 0.15}"/>
-      <geometry>
-        <box size="0.05 0.05 0.05"/>
-      </geometry>
-      <material name="blue">
-        <color rgba="0.2 0.2 0.8 1.0"/>
-      </material>
-    </visual>
-    <inertial>
-      <mass value="0.2"/>
-      <inertia ixx="0.001" ixy="0" ixz="0" iyy="0.001" iyz="0" izz="0.001"/>
-    </inertial>
-  </link>
-  <!-- Joints -->
-  <joint name="left_wheel_joint" type="continuous">
-    <origin xyz="0 ${wheel_sep/2} ${wheel_radius}" rpy="0 0 0"/>
-    <parent link="base_link"/>
-    <child link="left_wheel"/>
-    <axis xyz="0 1 0"/>
-  </joint>
-  <joint name="right_wheel_joint" type="continuous">
-    <origin xyz="0 -${wheel_sep/2} ${wheel_radius}" rpy="0 0 0"/>
-    <parent link="base_link"/>
-    <child link="right_wheel"/>
-    <axis xyz="0 1 0"/>
-  </joint>
-  <joint name="camera_joint" type="fixed">
-    <origin xyz="${chassis_length/2 - 0.1} 0 ${chassis_height + 0.15}"/>
-    <parent link="base_link"/>
-    <child link="camera_link"/>
-  </joint>
-  <!-- Gazebo plugins -->
-  <gazebo>
-    <plugin name="diff_drive" filename="libgazebo_ros_diff_drive.so">
-      <ros>
-        <namespace>/</namespace>
-      </ros>
-      <update_rate>50</update_rate>
-      <left_joint>left_wheel_joint</left_joint>
-      <right_joint>right_wheel_joint</right_joint>
-      <wheel_separation>${wheel_sep}</wheel_separation>
-      <wheel_diameter>${2*wheel_radius}</wheel_diameter>
-      <robot_base_frame>base_link</robot_base_frame>
-      <odom_topic>odom</odom_topic>
-      <command_topic>cmd_vel</command_topic>
-      <publish_tf>true</publish_tf>
-      <publish_odometry>true</publish_odometry>
-    </plugin>
-  </gazebo>
-  <!-- Camera sensor with Gazebo plugin -->
-  <gazebo reference="camera_link">
-    <sensor type="camera" name="camera_sensor">
-      <update_rate>15</update_rate>
-      <camera name="head_camera">
-        <horizontal_fov>1.047</horizontal_fov>
-        <image>
-          <width>640</width>
-          <height>480</height>
-          <format>R8G8B8</format>
-        </image>
-        <clip>
-          <near>0.05</near>
-          <far>20.0</far>
-        </clip>
-      </camera>
-      <plugin name="gazebo_ros_camera" filename="libgazebo_ros_camera.so">
-        <ros>
-          <namespace>/</namespace>
-        </ros>
-        <frame_name>camera_link</frame_name>
-        <camera_name>farm_camera</camera_name>
-        <image_topic_name>image_raw</image_topic_name>
-      </plugin>
-    </sensor>
-  </gazebo>
-</robot>
+/home/rutha/Projects/class_projects/robotics_final/src/farm_robot_description/urdf/farm_bot.xacro

File: src/farm_robot_description/urdf/farm_bot.xacro (robot description, xacro)
@@ -8,4 +8,6 @@
   <xacro:property name="chassis_height" value="0.12"/>
   <xacro:property name="wheel_sep" value="${chassis_width}"/>
+  <!-- Dummy root frame (avoids KDL root inertia issue) -->
+  <link name="base_footprint"/>
   <!-- Base link -->
   <link name="base_link">
@@ -91,4 +93,9 @@
   </link>
   <!-- Joints -->
+  <joint name="base_footprint_joint" type="fixed">
+    <origin xyz="0 0 0" rpy="0 0 0"/>
+    <parent link="base_footprint"/>
+    <child link="base_link"/>
+  </joint>
   <joint name="left_wheel_joint" type="continuous">
     <origin xyz="0 ${wheel_sep/2} ${wheel_radius}" rpy="0 0 0"/>
@@ -108,4 +115,51 @@
     <child link="camera_link"/>
   </joint>
+  <!-- Lidar Link -->
+  <link name="lidar_link">
+    <visual>
+      <geometry>
+        <cylinder radius="0.05" length="0.05"/>
+      </geometry>
+      <material name="black">
+        <color rgba="0 0 0 1"/>
+      </material>
+    </visual>
+  </link>
+  <joint name="lidar_joint" type="fixed">
+    <origin xyz="${chassis_length/2 - 0.05} 0 ${chassis_height + 0.05}" rpy="0 0 0"/>
+    <parent link="base_link"/>
+    <child link="lidar_link"/>
+  </joint>
+  <!-- Lidar Sensor -->
+  <gazebo reference="lidar_link">
+    <sensor type="ray" name="lidar_sensor">
+      <pose>0 0 0 0 0 0</pose>
+      <visualize>false</visualize>
+      <update_rate>10</update_rate>
+      <ray>
+        <scan>
+          <horizontal>
+            <samples>360</samples>
+            <resolution>1</resolution>
+            <min_angle>-3.14</min_angle>
+            <max_angle>3.14</max_angle>
+          </horizontal>
+        </scan>
+        <range>
+          <min>0.10</min>
+          <max>10.0</max>
+          <resolution>0.01</resolution>
+        </range>
+      </ray>
+      <plugin name="gazebo_ros_ray_sensor" filename="libgazebo_ros_ray_sensor.so">
+        <ros>
+          <namespace>/</namespace>
+          <remapping>~/out:=scan</remapping>
+        </ros>
+        <output_type>sensor_msgs/LaserScan</output_type>
+        <frame_name>lidar_link</frame_name>
+      </plugin>
+    </sensor>
+  </gazebo>
   <!-- Gazebo plugins -->
   <gazebo>
@@ -119,9 +173,10 @@
       <wheel_separation>${wheel_sep}</wheel_separation>
       <wheel_diameter>${2*wheel_radius}</wheel_diameter>
-      <robot_base_frame>base_link</robot_base_frame>
-      <odom_topic>odom</odom_topic>
+      <robot_base_frame>base_footprint</robot_base_frame>
+      <odometry_frame>odom</odometry_frame>
       <command_topic>cmd_vel</command_topic>
-      <publish_tf>true</publish_tf>
-      <publish_odometry>true</publish_odometry>
+      <publish_odom>true</publish_odom>
+      <publish_odom_tf>true</publish_odom_tf>
+      <publish_wheel_tf>true</publish_wheel_tf>
     </plugin>
   </gazebo>
